File: anti-aliasing_filter.kicad_pcb (KiCad board)
At the start: 2 copper layers, 16.5 x 21.6 mm, 11 parts, among them IC1 MCP6022, P1 CONN_4, P2 CONN_3

Commit message: Change R/C values to make 50kHz LP Chebychev
Parts:
- C1: value 0.0027uF -> 0.0047uF
- C2, C4: value 330pF -> 220pF
- R1: value 3.65k -> 1.78k
- R2: value 8.66k -> 4.02k
- R3: value 13.3k -> 9.09k
- R4: value 16.2k -> 20k
Changed lines of the file:
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@@
     (pad_to_mask_clearance 0)
     (aux_axis_origin 0 0)
-    (visible_elements FFFFF7BF)
+    (visible_elements 7FFFFFFF)
     (pcbplotparams
       (layerselection 284196865)
@@
       (effects (font (size 0.762 0.762) (thickness 0.127)))
     )
-    (fp_text value 3.65k (at 0 0) (layer F.SilkS) hide
+    (fp_text value 1.78k (at 0 0) (layer F.SilkS) hide
       (effects (font (size 0.762 0.762) (thickness 0.127)))
     )
@@
       (effects (font (size 0.762 0.762) (thickness 0.127)))
     )
-    (fp_text value 8.66k (at 0 0) (layer F.SilkS) hide
+    (fp_text value 4.02k (at 0 0) (layer F.SilkS) hide
       (effects (font (size 0.762 0.762) (thickness 0.127)))
     )
@@
       (effects (font (size 0.762 0.762) (thickness 0.127)))
     )
-    (fp_text value 330pF (at 0 0 180) (layer F.SilkS) hide
+    (fp_text value 220pF (at 0 0 180) (layer F.SilkS) hide
       (effects (font (size 0.762 0.762) (thickness 0.127)))
     )
@@
       (effects (font (size 0.762 0.762) (thickness 0.127)))
     )
-    (fp_text value 0.0027uF (at 0 0) (layer F.SilkS) hide
+    (fp_text value 0.0047uF (at 0 0) (layer F.SilkS) hide
       (effects (font (size 0.762 0.762) (thickness 0.127)))
     )
@@
       (effects (font (size 0.762 0.762) (thickness 0.127)))
     )
-    (fp_text value 13.3k (at 0 0 180) (layer F.SilkS) hide
+    (fp_text value 9.09k (at 0 0 180) (layer F.SilkS) hide
       (effects (font (size 0.762 0.762) (thickness 0.127)))
     )
@@
       (effects (font (size 0.762 0.762) (thickness 0.127)))
     )
-    (fp_text value 16.2k (at 0 0 180) (layer F.SilkS) hide
+    (fp_text value 20k (at 0 0 180) (layer F.SilkS) hide
       (effects (font (size 0.762 0.762) (thickness 0.127)))
     )
@@
       (effects (font (size 0.762 0.762) (thickness 0.127)))
     )
-    (fp_text value 330pF (at 0 0 180) (layer F.SilkS) hide
-      (effects (font (size 0.762 0.762) (thickness 0.127)))
-    )
+    (fp_text value 220pF (at 0 0 180) (layer F.SilkS) hide
+      (effects (font (size 0.762 0.762) (thickness 0.127)))
+    )
